File: ADC.sch (KiCad schematic (older format))
At the start: 76 parts

Commit message: schematics done
Parts:
- gave numbers to parts that had none: 60
Connections:
- net -1.25V_REF_BUF: now also U16.4; no longer U16.2
- net GNDA: now also U11.7, U15.2, U15.8; no longer U11.5, U15.4, U15.6
- net at C44.2, U14.2 (-), U16.1: now also U16.5; no longer U16.7
- net at C42.2, U12.2 (-), U16.7: now also U15.3; no longer U15.1
- net at JP6.1, U12.6 (-), U12.7: now also U15.6; no longer U15.8
- net at C43.1, JP10.1, U13.1: now also U16.3; no longer U16.4
- net at C43.2, U13.2 (-): now also U15.4, U16.6; no longer U15.3, U16.5
- net at JP7.1, U13.6 (-), U13.7: now also U15.5; no longer U15.6
- net at C39.1, U14.3 (+): now also U15.1, U15.7; no longer U15.3, U15.5
- net at C38.2, U14.5 (+): now also U11.2, U11.4; no longer U11.3, U11.4
- net at U11.1: now also U11.3; no longer U11.2
- new net: JP1.1, U11.5, U11.6

Commit message: board routed
ready for production
Parts:
- renumbered U16 to U15, U15 to U16
Connections:
- net +1.25V_REF_BUF: now also U15.6; no longer U16.8
- net -1.25V_REF_BUF: now also U15.5; no longer U15.4
- net GNDA: now also U15.7; no longer U15.2
- net at C44.2, U14.2 (-): now also U15.3, U15.4; no longer U15.5, U16.1
- net at C42.2, U12.2 (-), U16.7: now also U16.8; no longer U15.3
- net at JP6.1, U12.6 (-), U12.7: now also U16.1; no longer U15.6
- net at C43.2, U13.2 (-), U16.6: now also U16.5; no longer U16.4
- net at JP7.1, U13.6 (-), U13.7: now also U16.4; no longer U16.5
- net at C39.1, U14.3 (+), U15.1: now also U15.2; no longer U15.7
Other:
- moved on the sheet: C49, C50, C51, U12C, U13C, U14C
