File: DAC.sch (KiCad schematic (older format))
At the start: 21 parts

Commit message: schematics done
Parts:
- gave numbers to parts that had none: 16
Other:
- moved on the sheet: C34

Commit message: board routed
ready for production
Parts:
- removed C36: 1u, Capacitor_SMD:C_0603_1608Metric_Pad1.05x0.95mm_HandSolder, symbol Device:C
Connections:
- net GND: now also C37.2
- net GNDA: no longer C37.2
Changed lines of the file:
@@
 $EndComp
-Wire Wire Line
-	8350 2200 8350 2300
 Wire Wire Line
 	8650 2200 8650 2300
@@
 Connection ~ 7900 2300
 $Comp
-L Device:C C36
-U 1 1 5F9CD70C
-P 8500 2500
-F 0 "C36" H 8500 2600 50  0000 L CNN
-F 1 "1u" H 8500 2400 50  0000 L CNN
-F 2 "Capacitor_SMD:C_0603_1608Metric_Pad1.05x0.95mm_HandSolder" H 8538 2350 50  0001 C CNN
-F 3 "~" H 8500 2500 50  0001 C CNN
-	1    8500 2500
-	1    0    0    -1
-$EndComp
-$Comp
 L Device:C C37
 U 1 1 5F9CDB33
@@
 	1    0    0    -1
 $EndComp
-$Comp
-L power:GNDA #PWR083
-U 1 1 5F9CDF03
-P 8500 2700
-F 0 "#PWR083" H 8500 2450 50  0001 C CNN
-F 1 "GNDA" H 8505 2527 50  0000 C CNN
-F 2 "" H 8500 2700 50  0001 C CNN
-F 3 "" H 8500 2700 50  0001 C CNN
-	1    8500 2700
-	1    0    0    -1
-$EndComp
-$Comp
-L power:GNDA #PWR085
-U 1 1 5F9CE3DB
+Wire Wire Line
+	8800 2300 8800 2350
+Connection ~ 8800 2300
+Wire Wire Line
+	8800 2300 9700 2300
+Wire Wire Line
+	8800 2650 8800 2700
+Wire Wire Line
+	7750 2900 7850 2900
+Connection ~ 7750 2900
+Wire Wire Line
+	7750 2200 7750 2300
+Wire Wire Line
+	7750 2300 7900 2300
+Connection ~ 7750 2300
+Wire Wire Line
+	7750 2300 7750 2900
+Wire Wire Line
+	8350 2200 8350 2950
+$Comp
+L power:GND #PWR0122
+U 1 1 5F97239F
 P 8800 2700
-F 0 "#PWR085" H 8800 2450 50  0001 C CNN
-F 1 "GNDA" H 8805 2527 50  0000 C CNN
+F 0 "#PWR0122" H 8800 2450 50  0001 C CNN
+F 1 "GND" H 8805 2527 50  0000 C CNN
 F 2 "" H 8800 2700 50  0001 C CNN
 F 3 "" H 8800 2700 50  0001 C CNN
@@
 	1    0    0    -1
 $EndComp
-Wire Wire Line
-	8350 2300 8500 2300
-Wire Wire Line
-	8500 2300 8500 2350
-Connection ~ 8350 2300
-Wire Wire Line
-	8350 2300 8350 2950
-Wire Wire Line
-	8800 2300 8800 2350
-Connection ~ 8800 2300
-Wire Wire Line
-	8800 2300 9700 2300
-Wire Wire Line
-	8500 2650 8500 2700
-Wire Wire Line
-	8800 2650 8800 2700
-Wire Wire Line
-	7750 2900 7850 2900
-Connection ~ 7750 2900
-Wire Wire Line
-	7750 2200 7750 2300
-Wire Wire Line
-	7750 2300 7900 2300
-Connection ~ 7750 2300
-Wire Wire Line
-	7750 2300 7750 2900
 $EndSCHEMATC
