File: converters_1.sch (KiCad schematic (older format))
At the start: 1 part

Commit message: schematics done
Parts:
- added C1, C2, C22, C28: 6.8u 25V, Capacitor_SMD:CP_Elec_6.3x5.9, symbol Device:CP_Small
- added C10, C11, C12, C13, C14, C15, C16, C21, C23, C24, C25, C26, C27, C5, C6, C7, C8, C9: 1u, Capacitor_SMD:C_0603_1608Metric_Pad1.05x0.95mm_HandSolder, symbol Device:C_Small
- added C17, C18, C19, C20, C3, C4: 56u 25V, Capacitor_SMD:CP_Elec_6.3x5.9, symbol Device:CP_Small
- added D1, D10, D2, D3, D4, D5, D6, D7, D8, D9: BAT54WFILMY, Package_TO_SOT_SMD:SOT-323_SC-70, symbol Diode:BAT54W
- added H1, H2, H3, H4: MountingHole_Pad, MountingHole:MountingHole_3.2mm_M3_Pad_Via, symbol Mechanical:MountingHole_Pad
- added J1: +15V, MountingHole:MountingHole_2.2mm_M2_Pad_Via, symbol Connector:Conn_01x01_Male
- added J10, J11, J12, J9: Conn_01x10, Connector_PinHeader_2.54mm:PinHeader_1x10_P2.54mm_Vertical, symbol Connector_Generic:Conn_01x10
- added J13, J14, J15, J16, J7, J8: Conn_01x02, Connector_PinHeader_2.54mm:PinHeader_1x02_P2.54mm_Vertical, symbol Connector_Generic:Conn_01x02
- added J17: REF, MountingHole:MountingHole_2.2mm_M2_Pad_Via, symbol Connector:Conn_01x01_Male
- added J18, J19, J22, J24: AGND, MountingHole:MountingHole_2.2mm_M2_Pad_Via, symbol Connector:Conn_01x01_Male
- added J2: GND, MountingHole:MountingHole_2.2mm_M2_Pad_Via, symbol Connector:Conn_01x01_Male
- added J20: DAC_OUT, MountingHole:MountingHole_2.2mm_M2_Pad_Via, symbol Connector:Conn_01x01_Male
- added J21: ADC2, MountingHole:MountingHole_2.2mm_M2_Pad_Via, symbol Connector:Conn_01x01_Male
- added J23: ADC1, MountingHole:MountingHole_2.2mm_M2_Pad_Via, symbol Connector:Conn_01x01_Male
- added J3: -15V, MountingHole:MountingHole_2.2mm_M2_Pad_Via, symbol Connector:Conn_01x01_Male
- added J4, J5, J6: Conn_01x03, Connector_PinHeader_2.54mm:PinHeader_1x03_P2.54mm_Vertical, symbol Connector_Generic:Conn_01x03
- added R1, R11, R12, R14, R15, R2, R5, R6, R7, R8: 20k 1%, Resistor_SMD:R_0603_1608Metric_Pad1.05x0.95mm_HandSolder, symbol Device:R_Small
- added R10, R16, R3, R4, R9: ?, Resistor_SMD:R_0603_1608Metric_Pad1.05x0.95mm_HandSolder, symbol Device:R_Small
- added R13: 470k 1%, Resistor_SMD:R_0603_1608Metric_Pad1.05x0.95mm_HandSolder, symbol Device:R_Small
- added R17: 1k 1%, Resistor_SMD:R_0603_1608Metric_Pad1.05x0.95mm_HandSolder, symbol Device:R_Small
- added RV1: 10k, Potentiometer_THT:Potentiometer_Vishay_T73XW_Horizontal, symbol Device:R_POT_Small
- added TP1, TP10, TP11, TP2, TP3, TP4, TP5, TP6, TP7, TP8, TP9: TestPoint, TestPoint:TestPoint_Keystone_5010-5014_Multipurpose, symbol Connector:TestPoint
- added U1, U3, U6: LM317EMPX/NOPB, Package_TO_SOT_SMD:SOT-223-3_TabPin2, symbol Regulator_Linear:LM317_3PinPackage
- added U2, U4: LM337_SOT223, Package_TO_SOT_SMD:SOT-223-3_TabPin2, symbol Regulator_Linear:LM337_SOT223
- added U7: OPA333AID, Package_SO:SOIC-8_3.9x4.9mm_P1.27mm, symbol Amplifier_Operational:OPA333xxD
- gave numbers to parts that had none: 1
Connections:
- net +6V: now reaches U5.2 (VIN)
- net +6V: now also C1.1, C16.2, C19.1, C21.1, C5.2, D1.3 (K), D3.1 (A), D7.3 (K), J6.1 (Pin_1), R7.1, TP4.1, U1.3 (VI), U3.2 (VO)
- net at U5.3 (TEMP): now also U7.3 (+)
- net GNDA: now reaches U5.4 (GND)
- net GNDA: now also C1.2, C10.2, C11.1, C12.2, C13.2, C14.2, C15.1, C16.1, C17.2, C18.1, C19.2, C2.1, C20.1, C21.2, C24.2, C5.1, C6.2, C9.1, J13.1 (Pin_1), J14.1 (Pin_1), J15.1 (Pin_1), J16.2 (Pin_2), J18.1 (Pin_1), J19.1 (Pin_1), J22.1 (Pin_1), J24.1 (Pin_1), J5.2 (Pin_2), J6.2 (Pin_2), R10.1, R17.1, R3.2, R4.1, R9.2, TP5.1, TP6.1
- net at U5.5 (TRIM/NR): now also C24.1, R13.1
- net +5V_REF: now reaches U5.6 (VOUT)
- net +5V_REF: now also J15.2 (Pin_2), J17.1 (Pin_1), RV1.1, TP7.1
- new net: C11.2, D7.1 (A), R8.2, R9.1, U3.1 (ADJ)
- new net: C12.1, D8.3 (K), R10.2, R11.1, U4.1 (ADJ)
- new net: R7.2, R8.1
- new net: R13.2, RV1.2
- new net: R17.2, RV1.3
- new net: R11.2, R12.1
- new net: J8.1 (Pin_1), U7.2 (-), U7.6
- new net: C9.2, D5.1 (A), R2.2, R3.1, U1.1 (ADJ)
- new net: C10.1, D6.3 (K), R4.2, R5.1, U2.1 (ADJ)
- new net: R1.2, R2.1
- new net: R5.2, R6.1
- new net: C25.2, D10.1 (A), R15.2, R16.1, U6.1 (ADJ)
- new net: R14.2, R15.1
- new net +15V: C22.1, C23.2, C3.1, C7.2, D3.3 (K), D9.3 (K), J1.1 (Pin_1), J4.1 (Pin_1), U3.3 (VI), U6.3 (VI)
- new net +2V5: C15.2, C17.1, D1.1 (A), D5.3 (K), J5.1 (Pin_1), R1.1, TP3.1, U1.2 (VO)
- new net +3V3: C26.2, C27.2, C28.1, D10.3 (K), D9.1 (A), J10.10 (Pin_10), J11.10 (Pin_10), J12.10 (Pin_10), J7.1 (Pin_1), J9.10 (Pin_10), R14.1, TP8.1, U6.2 (VO), U7.7 (V+)
- new net -15V: C4.2, C8.1, D4.1 (A), J3.1 (Pin_1), J4.3 (Pin_3), U4.2 (VI)
- new net -2V5: C13.1, C18.2, D2.3 (K), D6.1 (A), J5.3 (Pin_3), R6.2, TP1.1, U2.3 (VO)
- new net -6V: C14.1, C2.2, C20.2, C6.1, D2.1 (A), D4.3 (K), D8.1 (A), J6.3 (Pin_3), R12.2, TP2.1, U2.2 (VI), U4.3 (VO)
- new net ADC/ADC_IN_1: J14.2 (Pin_2), J23.1 (Pin_1), TP11.1
- new net ADC/ADC_IN_2: J13.2 (Pin_2), J21.1 (Pin_1), TP10.1
- new net ADC/DIN: J10.3 (Pin_3), J12.3 (Pin_3)
- new net ADC/DOUT: J10.2 (Pin_2), J12.2 (Pin_2)
- new net ADC/SCLK: J10.4 (Pin_4), J12.4 (Pin_4)
- new net ADC/~CS: J10.5 (Pin_5), J12.5 (Pin_5)
- new net ADC/~DONE: J10.7 (Pin_7), J12.7 (Pin_7)
- new net ADC/~DRDY: J10.6 (Pin_6), J12.6 (Pin_6)
- new net ADC/~RESET: J10.8 (Pin_8), J12.8 (Pin_8)
- new net DAC/DAC_OUT: J16.1 (Pin_1), J20.1 (Pin_1), TP9.1
- new net DAC/SCLK: J11.8 (Pin_8), J9.8 (Pin_8)
- new net DAC/SDIN: J11.6 (Pin_6), J9.6 (Pin_6)
- new net DAC/SDO: J11.7 (Pin_7), J9.7 (Pin_7)
- new net DAC/~ALARM: J11.3 (Pin_3), J9.3 (Pin_3)
- new net DAC/~CLR: J11.4 (Pin_4), J9.4 (Pin_4)
- new net DAC/~LDAC: J11.2 (Pin_2), J9.2 (Pin_2)
- new net DAC/~SYNC: J11.5 (Pin_5), J9.5 (Pin_5)
- new net GND: C22.2, C23.1, C25.1, C26.1, C27.1, C28.2, C3.2, C4.1, C7.1, C8.2, H1.1, H2.1, H3.1, H4.1, J10.1 (Pin_1), J10.9 (Pin_9), J11.1 (Pin_1), J11.9 (Pin_9), J12.1 (Pin_1), J12.9 (Pin_9), J2.1 (Pin_1), J4.2 (Pin_2), J7.2 (Pin_2), J8.2 (Pin_2), J9.1 (Pin_1), J9.9 (Pin_9), R16.2, U7.4 (V-)
Other:
- note added: "V = 509 mV + 2.64 mV * T (C)"
- moved on the sheet: U5

Commit message: board routed
ready for production
Parts:
- removed C1, C2: 6.8u 25V, Capacitor_SMD:CP_Elec_6.3x5.9, symbol Device:CP_Small
- added D11, D12: G, LED_SMD:LED_0603_1608Metric_Pad1.05x0.95mm_HandSolder, symbol Device:LED
- added R36, R37: 20k 1%, Resistor_SMD:R_0603_1608Metric_Pad1.05x0.95mm_HandSolder, symbol Device:R_Small
Connections:
- net +15V: now also R36.1
- net -15V: now also D12.1 (K)
- net GND: now also D11.1 (K), R37.1
- new net: D12.2 (A), R37.2
- new net: D11.2 (A), R36.2
Changed lines of the file:
@@
 	-1   0    0    1
-$EndComp
-$Comp
-L Device:CP_Small C1
-U 1 1 5FA0FFC8
-P 650 1250
-F 0 "C1" H 738 1296 50  0000 L CNN
-F 1 "6.8u 25V" H 738 1205 50  0000 L CNN
-F 2 "Capacitor_SMD:CP_Elec_6.3x5.9" H 650 1250 50  0001 C CNN
-F 3 "~" H 650 1250 50  0001 C CNN
-	1    650  1250
-	1    0    0    -1
 $EndComp
 Wire Wire Line
 	1350 1050 1200 1050
-Wire Wire Line
-	650  1050 650  1150
 Connection ~ 1350 1050
 Wire Wire Line
@@
 	1200 1050 650  1050
 Wire Wire Line
-	650  1400 650  1350
-Wire Wire Line
 	1200 1400 1200 1350
 Wire Wire Line
 	650  950  650  1050
-Connection ~ 650  1050
 $Comp
 L Device:R_Small R1
@@
 	2150 3500 2050 3500
 $Comp
-L Device:CP_Small C2
-U 1 1 5FA10055
-P 650 3300
-F 0 "C2" H 738 3346 50  0000 L CNN
-F 1 "6.8u 25V" H 738 3255 50  0000 L CNN
-F 2 "Capacitor_SMD:CP_Elec_6.3x5.9" H 650 3300 50  0001 C CNN
-F 3 "~" H 650 3300 50  0001 C CNN
-	1    650  3300
-	1    0    0    -1
-$EndComp
-$Comp
 L Device:C_Small C?
 U 1 1 5FA1005B
@@
 $EndComp
 Wire Wire Line
-	650  3400 650  3500
-Wire Wire Line
 	650  3500 1200 3500
 Connection ~ 1350 3500
@@
 	1200 3500 1350 3500
 Wire Wire Line
-	650  3100 650  3200
-Wire Wire Line
 	1200 3100 1200 3200
 Wire Wire Line
 	650  3600 650  3500
-Connection ~ 650  3500
 $Comp
 L Diode:BAT54W D6
@@
 $EndComp
 $Comp
-L power:GNDA #PWR03
-U 1 1 5FA52331
-P 650 3100
-F 0 "#PWR03" H 650 2850 50  0001 C CNN
-F 1 "GNDA" H 655 2927 50  0000 C CNN
-F 2 "" H 650 3100 50  0001 C CNN
-F 3 "" H 650 3100 50  0001 C CNN
-	1    650  3100
-	-1   0    0    1
-$EndComp
-$Comp
 L power:GNDA #PWR013
 U 1 1 5FA536C6
@@
 F 3 "" H 1200 1400 50  0001 C CNN
 	1    1200 1400
-	1    0    0    -1
-$EndComp
-$Comp
-L power:GNDA #PWR02
-U 1 1 5FA5CEBF
-P 650 1400
-F 0 "#PWR02" H 650 1150 50  0001 C CNN
-F 1 "GNDA" H 655 1227 50  0000 C CNN
-F 2 "" H 650 1400 50  0001 C CNN
-F 3 "" H 650 1400 50  0001 C CNN
-	1    650  1400
 	1    0    0    -1
 $EndComp
@@
 	1    0    0    -1
 $EndComp
+$Comp
+L Device:LED D12
+U 1 1 5F912F6B
+P 4150 6200
+F 0 "D12" V 4189 6082 50  0000 R CNN
+F 1 "G" V 4098 6082 50  0000 R CNN
+F 2 "LED_SMD:LED_0603_1608Metric_Pad1.05x0.95mm_HandSolder" H 4150 6200 50  0001 C CNN
+F 3 "~" H 4150 6200 50  0001 C CNN
+	1    4150 6200
+	0    -1   -1   0
+$EndComp
+$Comp
+L Device:R_Small R36
+U 1 1 5F91618A
+P 4150 5150
+F 0 "R36" H 4209 5196 50  0000 L CNN
+F 1 "20k 1%" H 4209 5105 50  0000 L CNN
+F 2 "Resistor_SMD:R_0603_1608Metric_Pad1.05x0.95mm_HandSolder" H 4150 5150 50  0001 C CNN
+F 3 "~" H 4150 5150 50  0001 C CNN
+	1    4150 5150
+	1    0    0    -1
+$EndComp
+$Comp
+L Device:R_Small R37
+U 1 1 5F917692
+P 4150 5850
+F 0 "R37" H 4209 5896 50  0000 L CNN
+F 1 "20k 1%" H 4209 5805 50  0000 L CNN
+F 2 "Resistor_SMD:R_0603_1608Metric_Pad1.05x0.95mm_HandSolder" H 4150 5850 50  0001 C CNN
+F 3 "~" H 4150 5850 50  0001 C CNN
+	1    4150 5850
+	1    0    0    -1
+$EndComp
+$Comp
+L power:+15V #PWR0120
+U 1 1 5F91814F
+P 4150 5000
+F 0 "#PWR0120" H 4150 4850 50  0001 C CNN
+F 1 "+15V" H 4165 5173 50  0000 C CNN
+F 2 "" H 4150 5000 50  0001 C CNN
+F 3 "" H 4150 5000 50  0001 C CNN
+	1    4150 5000
+	1    0    0    -1
+$EndComp
+$Comp
+L power:-15V #PWR0121
+U 1 1 5F91887A
+P 4150 6400
+F 0 "#PWR0121" H 4150 6500 50  0001 C CNN
+F 1 "-15V" H 4150 6550 50  0000 C CNN
+F 2 "" H 4150 6400 50  0001 C CNN
+F 3 "" H 4150 6400 50  0001 C CNN
+	1    4150 6400
+	-1   0    0    1
+$EndComp
+Wire Wire Line
+	4150 6400 4150 6350
+Wire Wire Line
+	4150 6050 4150 5950
+$Comp
+L Device:LED D11
+U 1 1 5F91489E
+P 4150 5500
+F 0 "D11" V 4189 5382 50  0000 R CNN
+F 1 "G" V 4098 5382 50  0000 R CNN
+F 2 "LED_SMD:LED_0603_1608Metric_Pad1.05x0.95mm_HandSolder" H 4150 5500 50  0001 C CNN
+F 3 "~" H 4150 5500 50  0001 C CNN
+	1    4150 5500
+	0    -1   -1   0
+$EndComp
+Wire Wire Line
+	4150 5350 4150 5250
+Wire Wire Line
+	4150 5650 4150 5700
+Wire Wire Line
+	4150 5000 4150 5050
+$Comp
+L power:GND #PWR0119
+U 1 1 5F9C9A92
+P 3950 5800
+F 0 "#PWR0119" H 3950 5550 50  0001 C CNN
+F 1 "GND" H 3955 5627 50  0000 C CNN
+F 2 "" H 3950 5800 50  0001 C CNN
+F 3 "" H 3950 5800 50  0001 C CNN
+	1    3950 5800
+	1    0    0    -1
+$EndComp
+Wire Wire Line
+	3950 5800 3950 5700
+Wire Wire Line
+	3950 5700 4150 5700
+Connection ~ 4150 5700
+Wire Wire Line
+	4150 5700 4150 5750
 $EndSCHEMATC

Commit message: GND - AGND tie added
Parts:
- added NT1: GND TIE, NetTie:NetTie-2_SMD_Pad2.0mm, symbol Device:Net-Tie_2
Connections:
- net GND: now also NT1.1
- net GNDA: now also NT1.2
Changed lines of the file:
@@
 Wire Wire Line
 	4150 5700 4150 5750
+$Comp
+L Device:Net-Tie_2 NT1
+U 1 1 5F9BCD1E
+P 4050 4200
+F 0 "NT1" H 4050 4381 50  0000 C CNN
+F 1 "GND TIE" H 4050 4290 50  0000 C CNN
+F 2 "NetTie:NetTie-2_SMD_Pad2.0mm" H 4050 4200 50  0001 C CNN
+F 3 "~" H 4050 4200 50  0001 C CNN
+	1    4050 4200
+	1    0    0    -1
+$EndComp
+$Comp
+L power:GNDA #PWR?
+U 1 1 5F9BD8FE
+P 4200 4250
+F 0 "#PWR?" H 4200 4000 50  0001 C CNN
+F 1 "GNDA" H 4205 4077 50  0000 C CNN
+F 2 "" H 4200 4250 50  0001 C CNN
+F 3 "" H 4200 4250 50  0001 C CNN
+	1    4200 4250
+	1    0    0    -1
+$EndComp
+$Comp
+L power:GND #PWR?
+U 1 1 5F9BE238
+P 3900 4250
+F 0 "#PWR?" H 3900 4000 50  0001 C CNN
+F 1 "GND" H 3905 4077 50  0000 C CNN
+F 2 "" H 3900 4250 50  0001 C CNN
+F 3 "" H 3900 4250 50  0001 C CNN
+	1    3900 4250
+	1    0    0    -1
+$EndComp
+Wire Wire Line
+	3900 4250 3900 4200
+Wire Wire Line
+	3900 4200 3950 4200
+Wire Wire Line
+	4150 4200 4200 4200
+Wire Wire Line
+	4200 4200 4200 4250
 $EndSCHEMATC
